Commit message: 修复go2安装

File: robots/go1_description/xacro/go1.champ.urdf (robot description, URDF)
Before this commit: robot go1_description, 38 links, 37 joints
Links:
- added link velodyne, mass 0.01; visual mesh filename=package://velodyne_description/meshes/VLP16_scan.dae
- added link velodyne_base_link, mass 0.83; collision cylinder length=0.0717 radius=0.0516; visual mesh filename=package://velodyne_description/meshes/VLP16_base_1.dae
Joints:
- added joint velodyne_base_mount_joint: type fixed, parent trunk, child velodyne_base_link, origin xyz=0 0 0.08 rpy=0 0 0
- added joint velodyne_base_scan_joint: type fixed, parent velodyne_base_link, child velodyne, origin xyz=0 0 0.0377 rpy=0 0 0
